File: mainboard.sch (KiCad schematic (older format))
At the start: 7 parts

Commit message: Beta version
Parts:
- added C1, C2: C, Capacitors_SMD:C_0603, symbol C
- added C3: 10u, Capacitors_SMD:C_0603, symbol C
- added C4, C5, C6, C7: 0.1u, Capacitors_SMD:C_0603, symbol C
- added C8: CP, Capacitors_SMD:CP_Elec_5x5.8, symbol CP
- added D4: D, Diodes_SMD:D_SMA, symbol D
- added IC1: MCP25625-E_ML, MCP25625-E_ML:QFN65P600X600X100-29N-D, symbol MCP25625-E_ML
- added J1: SENS1, Connectors_JST:JST_PH_S3B-PH-SM4-TB_03x2.00mm_Angled, symbol Conn_01x03
- added J10: R4, Connectors_JST:JST_PH_S3B-PH-SM4-TB_03x2.00mm_Angled, symbol Conn_01x03
- added J11: R5, Connectors_JST:JST_PH_S3B-PH-SM4-TB_03x2.00mm_Angled, symbol Conn_01x03
- added J12: R6, Connectors_JST:JST_PH_S3B-PH-SM4-TB_03x2.00mm_Angled, symbol Conn_01x03
- added J13: SW1, Connectors_JST:JST_PH_S3B-PH-SM4-TB_03x2.00mm_Angled, symbol Conn_01x03
- added J14: SW2, Connectors_JST:JST_PH_S3B-PH-SM4-TB_03x2.00mm_Angled, symbol Conn_01x03
- added J15: SW3, Connectors_JST:JST_PH_S3B-PH-SM4-TB_03x2.00mm_Angled, symbol Conn_01x03
- added J16: SW4, Connectors_JST:JST_PH_S3B-PH-SM4-TB_03x2.00mm_Angled, symbol Conn_01x03
- added J17: SW5, Connectors_JST:JST_PH_S3B-PH-SM4-TB_03x2.00mm_Angled, symbol Conn_01x03
- added J18: SW6, Connectors_JST:JST_PH_S3B-PH-SM4-TB_03x2.00mm_Angled, symbol Conn_01x03
- added J19, J20, J21, J22, J26, J27: Conn_01x03, Connectors_JST:JST_PH_B3B-PH-K_03x2.00mm_Straight, symbol Conn_01x03
- added J2: SENS2, Connectors_JST:JST_PH_S3B-PH-SM4-TB_03x2.00mm_Angled, symbol Conn_01x03
- added J23, J24, J25: Screw_Terminal_01x02, Custom Connector:ZFKDS, symbol Screw_Terminal_01x02
- added J28, J31: Conn_01x04, Pin_Headers:Pin_Header_Straight_1x04_Pitch2.54mm, symbol Conn_01x04
- added J29: Conn_01x03, Connectors:GS3, symbol Conn_01x03
- added J3: SENS3, Connectors_JST:JST_PH_S3B-PH-SM4-TB_03x2.00mm_Angled, symbol Conn_01x03
- added J30: Screw_Terminal_01x03, TerminalBlocks_Phoenix:TerminalBlock_Phoenix_MPT-2.54mm_3pol, symbol Screw_Terminal_01x03
- added J32, J33: Conn_01x10, Pin_Headers:Pin_Header_Straight_1x09_Pitch2.54mm, symbol Conn_01x10
- added J4: SENS4, Connectors_JST:JST_PH_S3B-PH-SM4-TB_03x2.00mm_Angled, symbol Conn_01x03
- added J5: SENS5, Connectors_JST:JST_PH_S3B-PH-SM4-TB_03x2.00mm_Angled, symbol Conn_01x03
- added J6: SENS6, Connectors_JST:JST_PH_S3B-PH-SM4-TB_03x2.00mm_Angled, symbol Conn_01x03
- added J7: R1, Connectors_JST:JST_PH_S3B-PH-SM4-TB_03x2.00mm_Angled, symbol Conn_01x03
- added J8: R2, Connectors_JST:JST_PH_S3B-PH-SM4-TB_03x2.00mm_Angled, symbol Conn_01x03
- added J9: R3, Connectors_JST:JST_PH_S3B-PH-SM4-TB_03x2.00mm_Angled, symbol Conn_01x03
- added K1, K2, K3, K4, K5, K6: EE2-5NU, EE2-5NU, symbol EE2-5NU
- added Q1, Q2: DMP2100U, TO_SOT_Packages_SMD:SOT-23, symbol NTR2101P
- added R10, R12, R14, R16, R18, R20, R22, R24, R30, R31, R4, R6, R8: 4k7, Resistors_SMD:R_0603, symbol R
- added R11, R13, R15, R17, R19, R21, R23, R25, R26, R5, R7, R9: 330, Resistors_SMD:R_0603, symbol R
- added R27: 1K, Resistors_SMD:R_0603, symbol R
- added R28: 10k, Resistors_SMD:R_0603, symbol R
- added R29: 120, Resistors_SMD:R_0603, symbol R
- added SW1: SW_Push, Buttons_Switches_SMD:SW_SPST_EVQPE1, symbol SW_Push
- added U1: ULN2003A, Housings_SSOP:TSSOP-16-1EP_4.4x5mm_Pitch0.65mm, symbol ULN2003A
- added U2, U3, U4: LTV-847, Housings_DIP:DIP-16_W8.89mm_SMDSocket_LongPads, symbol LTV-847
- added U5: 74LS241, Housings_SOIC:SOIC-20W_7.5x12.8mm_Pitch1.27mm, symbol 74LS241
- added Y1: Crystal, symbol Crystal
- D1, D2, D3: footprint LEDs:LED_0805 -> LEDs:LED_0603
- R1, R3: value R -> 330; footprint Resistors_SMD:R_0805 -> Resistors_SMD:R_0603
- R2: value R -> 4k7; footprint Resistors_SMD:R_0805 -> Resistors_SMD:R_0603
Connections:
- net labels added: +12V, +5VA, A0, A1, A10, A11, A12, A13, A14, A15, A2, A3, A4, A5, A6, A7, A8, A9, AX_CONTROL, AX_RX, AX_SIGNAL, AX_TX, CANH, CANL, CAN_CS, CAN_INT, CAN_MISO, CAN_MOSI, CAN_SCK, C_RX, C_TX, DBG_RX, DBG_TX, PWM1, PWM2, PWM3, R1, R1_CONT, R1_SIG, R2, R2_CONT, R2_SIG, R3, R3_CONT, R3_SIG, R4, R4_CONT, R4_SIG, R5, R5_CONT, R5_SIG, R6, R6_CONT, R6_SIG, RST, SCL, SDA, SENS1, SENS2, SENS3, SENS4, SENS5, SENS6, SO_1, SO_2, SO_3, SO_4, SO_5, SO_6, SW1, SW2, SW3, SW4, SW5, SW6, SWO_1, SWO_2, SWO_3, SWO_4, SWO_5, SWO_6
- net labels removed: D13
- wire segments 14 -> 425
- no-connect marks 0 -> 45
Other:
- note added: "SENSOR"
- moved on the sheet: XA1

Commit message: Finished version 1.0
Parts:
- removed C1, C2: C, Capacitors_SMD:C_0603, symbol C
- removed C3: 10u, Capacitors_SMD:C_0603, symbol C
- removed C4, C5, C6, C7: 0.1u, Capacitors_SMD:C_0603, symbol C
- removed D1, D2, D3: LED, LEDs:LED_0603, symbol LED
- removed IC1: MCP25625-E_ML, MCP25625-E_ML:QFN65P600X600X100-29N-D, symbol MCP25625-E_ML
- removed J1: SENS1, Connectors_JST:JST_PH_S3B-PH-SM4-TB_03x2.00mm_Angled, symbol Conn_01x03
- removed J10: R4, Connectors_JST:JST_PH_S3B-PH-SM4-TB_03x2.00mm_Angled, symbol Conn_01x03
- removed J11: R5, Connectors_JST:JST_PH_S3B-PH-SM4-TB_03x2.00mm_Angled, symbol Conn_01x03
- removed J12: R6, Connectors_JST:JST_PH_S3B-PH-SM4-TB_03x2.00mm_Angled, symbol Conn_01x03
- removed J13: SW1, Connectors_JST:JST_PH_S3B-PH-SM4-TB_03x2.00mm_Angled, symbol Conn_01x03
- removed J14: SW2, Connectors_JST:JST_PH_S3B-PH-SM4-TB_03x2.00mm_Angled, symbol Conn_01x03
- removed J15: SW3, Connectors_JST:JST_PH_S3B-PH-SM4-TB_03x2.00mm_Angled, symbol Conn_01x03
- removed J16: SW4, Connectors_JST:JST_PH_S3B-PH-SM4-TB_03x2.00mm_Angled, symbol Conn_01x03
- removed J17: SW5, Connectors_JST:JST_PH_S3B-PH-SM4-TB_03x2.00mm_Angled, symbol Conn_01x03
- removed J18: SW6, Connectors_JST:JST_PH_S3B-PH-SM4-TB_03x2.00mm_Angled, symbol Conn_01x03
- removed J19, J20, J21, J22, J26, J27: Conn_01x03, Connectors_JST:JST_PH_B3B-PH-K_03x2.00mm_Straight, symbol Conn_01x03
- removed J2: SENS2, Connectors_JST:JST_PH_S3B-PH-SM4-TB_03x2.00mm_Angled, symbol Conn_01x03
- removed J23, J24, J25: Screw_Terminal_01x02, Custom Connector:ZFKDS, symbol Screw_Terminal_01x02
- removed J28, J31: Conn_01x04, Pin_Headers:Pin_Header_Straight_1x04_Pitch2.54mm, symbol Conn_01x04
- removed J29: Conn_01x03, Connectors:GS3, symbol Conn_01x03
- removed J3: SENS3, Connectors_JST:JST_PH_S3B-PH-SM4-TB_03x2.00mm_Angled, symbol Conn_01x03
- removed J30: Screw_Terminal_01x03, TerminalBlocks_Phoenix:TerminalBlock_Phoenix_MPT-2.54mm_3pol, symbol Screw_Terminal_01x03
- removed J32, J33: Conn_01x10, Pin_Headers:Pin_Header_Straight_1x09_Pitch2.54mm, symbol Conn_01x10
- removed J4: SENS4, Connectors_JST:JST_PH_S3B-PH-SM4-TB_03x2.00mm_Angled, symbol Conn_01x03
- removed J5: SENS5, Connectors_JST:JST_PH_S3B-PH-SM4-TB_03x2.00mm_Angled, symbol Conn_01x03
- removed J6: SENS6, Connectors_JST:JST_PH_S3B-PH-SM4-TB_03x2.00mm_Angled, symbol Conn_01x03
- removed J7: R1, Connectors_JST:JST_PH_S3B-PH-SM4-TB_03x2.00mm_Angled, symbol Conn_01x03
- removed J8: R2, Connectors_JST:JST_PH_S3B-PH-SM4-TB_03x2.00mm_Angled, symbol Conn_01x03
- removed J9: R3, Connectors_JST:JST_PH_S3B-PH-SM4-TB_03x2.00mm_Angled, symbol Conn_01x03
- removed K1, K2, K3, K4, K5, K6: EE2-5NU, EE2-5NU, symbol EE2-5NU
- removed Q2: DMP2100U, TO_SOT_Packages_SMD:SOT-23, symbol NTR2101P
- removed R1, R11, R13, R15, R17, R19, R21, R23, R25, R26, R3, R5, R7, R9: 330, Resistors_SMD:R_0603, symbol R
- removed R10, R12, R14, R16, R18, R2, R20, R22, R24, R4, R6, R8: 4k7, Resistors_SMD:R_0603, symbol R
- removed R27: 1K, Resistors_SMD:R_0603, symbol R
- removed R28: 10k, Resistors_SMD:R_0603, symbol R
- removed R29: 120, Resistors_SMD:R_0603, symbol R
- removed U2, U3, U4: LTV-847, Housings_DIP:DIP-16_W8.89mm_SMDSocket_LongPads, symbol LTV-847
- removed Y1: Crystal, symbol Crystal
- added C1, C10, C11, C12, C3, C7, C9: 100n, Capacitor_SMD:C_0603_1608Metric, symbol Device:C
- added C13: CP, Capacitor_SMD:CP_Elec_5x5.8, symbol mainboard-rescue:CP
- added C2, C4: 10u, Capacitor_SMD:C_0603_1608Metric, symbol Device:C
- added C5, C6: 20p, Capacitor_SMD:C_0603_1608Metric, symbol Device:C
- added D1, D2: D, Diode_SMD:D_SMA, symbol mainboard-rescue:D
- added D3, D5, D6, D7: LED, LED_SMD:LED_0603_1608Metric, symbol Device:LED
- added J1: Conn_01x10, Connector_PinHeader_1.27mm:PinHeader_1x10_P1.27mm_Vertical, symbol Connector_Generic:Conn_01x10
- added J10: jump_side, Connector_JST:JST_XH_B04B-XH-A_1x04_P2.50mm_Vertical, symbol Connector_Generic:Conn_01x04
- added J11: Senzor1, Connector_JST:JST_XH_B03B-XH-A_1x03_P2.50mm_Vertical, symbol mainboard-rescue:Conn_01x03
- added J12: tactics_sw, Connector_JST:JST_XH_B04B-XH-A_1x04_P2.50mm_Vertical, symbol Connector_Generic:Conn_01x04
- added J13: i2c_con, Connector_JST:JST_XH_B04B-XH-A_1x04_P2.50mm_Vertical, symbol Connector_Generic:Conn_01x04
- added J14: ser_con, Connector_JST:JST_XH_B03B-XH-A_1x03_P2.50mm_Vertical, symbol Connector_Generic:Conn_01x03
- added J15: CAN, Connector_JST:JST_XH_B03B-XH-A_1x03_P2.50mm_Vertical, symbol mainboard-rescue:Conn_01x03
- added J17: Senzor3, Connector_JST:JST_XH_B03B-XH-A_1x03_P2.50mm_Vertical, symbol mainboard-rescue:Conn_01x03
- added J18: Senzor5, Connector_JST:JST_XH_B03B-XH-A_1x03_P2.50mm_Vertical, symbol mainboard-rescue:Conn_01x03
- added J19: SERVO1, Connector_JST:JST_XH_B03B-XH-A_1x03_P2.50mm_Vertical, symbol Connector_Generic:Conn_01x03
- added J2: AX, Connector_JST:JST_XH_B04B-XH-A_1x04_P2.50mm_Vertical, symbol mainboard-rescue:Screw_Terminal_01x04
- added J20: SERVO2, Connector_JST:JST_XH_B03B-XH-A_1x03_P2.50mm_Vertical, symbol Connector_Generic:Conn_01x03
- added J21: S2, Connector_JST:JST_XH_B02B-XH-A_1x02_P2.50mm_Vertical, symbol mainboard-rescue:Screw_Terminal_01x02
- added J22: S3, Connector_JST:JST_XH_B02B-XH-A_1x02_P2.50mm_Vertical, symbol mainboard-rescue:Screw_Terminal_01x02
- added J23: 12V_IN, PHOENIX_1702473, symbol 1702473:1702473
- added J24: 5V_IN, PHOENIX_1702473, symbol 1702473:1702473
- added J25: 5VA_IN, PHOENIX_1702473, symbol 1702473:1702473
- added J26: S4, Connector_JST:JST_XH_B02B-XH-A_1x02_P2.50mm_Vertical, symbol mainboard-rescue:Screw_Terminal_01x02
- added J27: S5, Connector_JST:JST_XH_B02B-XH-A_1x02_P2.50mm_Vertical, symbol mainboard-rescue:Screw_Terminal_01x02
- added J28: S6, Connector_JST:JST_XH_B02B-XH-A_1x02_P2.50mm_Vertical, symbol mainboard-rescue:Screw_Terminal_01x02
- added J3: bin_sens1, Connector_JST:JST_XH_B03B-XH-A_1x03_P2.50mm_Vertical, symbol Connector_Generic:Conn_01x03
- added J30: Senzor2, Connector_JST:JST_XH_B03B-XH-A_1x03_P2.50mm_Vertical, symbol mainboard-rescue:Conn_01x03
- added J31: Senzor4, Connector_JST:JST_XH_B03B-XH-A_1x03_P2.50mm_Vertical, symbol mainboard-rescue:Conn_01x03
- added J32: Senzor6, Connector_JST:JST_XH_B03B-XH-A_1x03_P2.50mm_Vertical, symbol mainboard-rescue:Conn_01x03
- added J33: SERVO3, Connector_JST:JST_XH_B03B-XH-A_1x03_P2.50mm_Vertical, symbol Connector_Generic:Conn_01x03
- added J34: SERVO4, Connector_JST:JST_XH_B03B-XH-A_1x03_P2.50mm_Vertical, symbol Connector_Generic:Conn_01x03
- added J35: RELAY2, PHOENIX_1702473, symbol 1702473:1702473
- added J36: RELAY1, PHOENIX_1702473, symbol 1702473:1702473
- added J4: bin_sens4, Connector_JST:JST_XH_B03B-XH-A_1x03_P2.50mm_Vertical, symbol Connector_Generic:Conn_01x03
- added J5: S1, Connector_JST:JST_XH_B02B-XH-A_1x02_P2.50mm_Vertical, symbol mainboard-rescue:Screw_Terminal_01x02
- added J6: bin_sens2, Connector_JST:JST_XH_B03B-XH-A_1x03_P2.50mm_Vertical, symbol Connector_Generic:Conn_01x03
- added J7: bin_sens5, Connector_JST:JST_XH_B03B-XH-A_1x03_P2.50mm_Vertical, symbol Connector_Generic:Conn_01x03
- added J8: bin_sens3, Connector_JST:JST_XH_B03B-XH-A_1x03_P2.50mm_Vertical, symbol Connector_Generic:Conn_01x03
- added J9: bin_sens6, Connector_JST:JST_XH_B03B-XH-A_1x03_P2.50mm_Vertical, symbol Connector_Generic:Conn_01x03
- added K1, K2: G5Q-1A, Relay_THT:Relay_SPST_Omron-G5Q-1A, symbol Relay:G5Q-1A
- added Q2: DMP2100U, Package_TO_SOT_SMD:SOT-23, symbol mainboard-rescue:NTR2101P
- added R1, R11, R12, R13, R16, R18, R20, R22, R23, R24, R6, R8: 500, Resistor_SMD:R_0603_1608Metric, symbol mainboard-rescue:R
- added R10, R14, R15, R25, R26, R27, R5: 10K, Resistor_SMD:R_0603_1608Metric, symbol mainboard-rescue:R
- added R17, R19, R2, R21, R28, R29, R3, R33, R34, R7, R9: 1K, Resistor_SMD:R_0603_1608Metric, symbol mainboard-rescue:R
- added R32: 120, Resistor_SMD:R_0603_1608Metric, symbol mainboard-rescue:R
- added R4: 2K, Resistor_SMD:R_0603_1608Metric, symbol mainboard-rescue:R
- added U10, U11, U12, U2, U8, U9: PC817, Package_SO:SOP-4_4.4x2.8mm_P1.27mm, symbol mainboard-rescue:PC817
- added U3: NRF24L01_Breakout, Connector_PinHeader_2.54mm:PinHeader_2x04_P2.54mm_Vertical, symbol RF:NRF24L01_Breakout
- added U4: Bluetooth_HC-05, Bluetooth:Bluetooth_HC-05, symbol Bluetooth:Bluetooth_HC-05
- added U6: MCP25625-x-SS, Package_SO:SSOP-28_5.3x10.2mm_P0.65mm, symbol Interface_CAN_LIN:MCP25625-x-SS
- added U7: ULN2003A, Package_SO:TSSOP-16-1EP_4.4x5mm_P0.65mm, symbol mainboard-rescue:ULN2003A
- added Y1: Crystal_GND24, Crystal:Crystal_SMD_SeikoEpson_FA238V-4Pin_3.2x2.5mm_HandSoldering, symbol Device:Crystal_GND24
- C8: footprint Capacitors_SMD:CP_Elec_5x5.8 -> Capacitor_SMD:CP_Elec_5x5.8; symbol CP -> mainboard-rescue:CP
- D4: footprint Diodes_SMD:D_SMA -> Diode_SMD:D_SMA; symbol D -> mainboard-rescue:D
- Q1: footprint TO_SOT_Packages_SMD:SOT-23 -> Package_TO_SOT_SMD:SOT-23; symbol NTR2101P -> mainboard-rescue:NTR2101P
- R30, R31: footprint Resistors_SMD:R_0603 -> Resistor_SMD:R_0603_1608Metric; symbol R -> mainboard-rescue:R
- RESET1: renamed from SW1; footprint Buttons_Switches_SMD:SW_SPST_EVQPE1 -> Button_Switch_SMD:SW_SPST_FSMSM; symbol SW_Push -> mainboard-rescue:SW_Push
- U1: footprint Housings_SSOP:TSSOP-16-1EP_4.4x5mm_Pitch0.65mm -> Package_SO:TSSOP-16-1EP_4.4x5mm_P0.65mm; symbol ULN2003A -> mainboard-rescue:ULN2003A
- U5: footprint Housings_SOIC:SOIC-20W_7.5x12.8mm_Pitch1.27mm -> Package_SO:SOIC-20W_7.5x12.8mm_P1.27mm; symbol 74LS241 -> mainboard-rescue:74LS241
- XA1: symbol Arduino_Mega2560_Shield -> mainboard-rescue:Arduino_Mega2560_Shield
Connections:
- net labels added: AX_PWR, BIN_SEN1, BIN_SEN2, BIN_SEN3, BIN_SEN4, BIN_SEN5, BIN_SEN6, JUMPER, NRF_CE, NRF_CS, PWM4, SENSOR1, SENSOR2, SENSOR3, SENSOR4, SENSOR5, SENSOR6, SER_RX, SER_TX, SIDE, TACTIC1, TACTIC2, _S1, _S1_SIG, _S2, _S2_SIG, _S3, _S3_SIG, _S4, _S4_SIG, _S5, _S5_SIG, _S6, _S6_SIG
- net labels removed: A0, A1, A10, A11, A12, A13, A14, A15, A2, A3, A4, A5, A6, A7, A8, A9, CANH, CANL, C_RX, C_TX, R1, R2, R3, R3_CONT, R3_SIG, R4, R4_CONT, R4_SIG, R5, R5_CONT, R5_SIG, R6, R6_CONT, R6_SIG, SENS1, SENS2, SENS3, SENS4, SENS5, SENS6, SO_1, SO_2, SO_3, SO_4, SO_5, SO_6, SW1, SW2, SW3, SW4, SW5, SW6, SWO_1, SWO_2, SWO_3, SWO_4, SWO_5, SWO_6
- wire segments 425 -> 462
- no-connect marks 45 -> 51
Other:
- note added: "12V, 5VA, 5V Inputs with protection,\nLED indicators"
- note added: "4x servo"
- note added: "6x 12V sensors with isolation (PC817)"
- note added: "6x binary 5V switch connectors"
- note added: "AX-12 servo support"
- note added: "Arduino MEGA pinout"
- note added: "Control a low-current device (ON/OFF)\n(electric valve)"
- note added: "HC-05 Bluetooth module"
- note added: "Jumper, Side & Tactics connector\nCommunication connectors (I2C, Serial)"
- note added: "MCP25625 - CAN controller\nCAN 2.0 supported, up to 1Mbps\nWorking on 16MHz\n"
- note added: "Two high power relays (12V devices)"
- note added: "fit if necessary"
- note added: "nRF24L01"
- note removed: "SENSOR"
- moved on the sheet: C8, D4, Q1, R30, R31, RESET1, U1, U5, XA1

Commit message: Readme and images
Parts:
- J23, J24, J25, J35, J36: symbol 1702473:1702473 -> mainboard-rescue:1702473-1702473
- U4: symbol Bluetooth:Bluetooth_HC-05 -> mainboard-rescue:Bluetooth_HC-05-Bluetooth
Changed lines of the file:
@@
 EESchema Schematic File Version 4
 LIBS:mainboard-cache
-EELAYER 26 0
+EELAYER 29 0
 EELAYER END
 $Descr A3 16535 11693
@@
 	5950 8150 6000 8150
 $Comp
-L Bluetooth:Bluetooth_HC-05 U4
+L mainboard-rescue:Bluetooth_HC-05-Bluetooth U4
 U 1 1 5D18ACD6
 P 5650 1350
@@
 $EndComp
 $Comp
-L 1702473:1702473 J23
+L mainboard-rescue:1702473-1702473 J23
 U 1 1 5C2AB30F
 P 11300 7500
@@
 	12100 7700 12050 7700
 $Comp
-L 1702473:1702473 J24
+L mainboard-rescue:1702473-1702473 J24
 U 1 1 5C4121AE
 P 10000 7450
@@
 $EndComp
 $Comp
-L 1702473:1702473 J25
+L mainboard-rescue:1702473-1702473 J25
 U 1 1 5C6EBC8F
 P 8750 7450
@@
 $EndComp
 $Comp
-L 1702473:1702473 J35
+L mainboard-rescue:1702473-1702473 J35
 U 1 1 5C886E21
 P 4250 4750
@@
 $EndComp
 $Comp
-L 1702473:1702473 J36
+L mainboard-rescue:1702473-1702473 J36
 U 1 1 5CA93910
 P 5450 4750
@@
 F 1 "Crystal_GND24" V 7050 8550 50  0000 L CNN
 F 2 "Crystal:Crystal_SMD_SeikoEpson_FA238V-4Pin_3.2x2.5mm_HandSoldering" H 7350 8700 50  0001 C CNN
-F 3 "https://www.digikey.com/product-detail/en/ecs-inc/ECS-160-20-3X-TR/XC1776CT-ND/2676640" H 7350 8700 50  0001 C CNN
+F 3 "" H 7350 8700 50  0001 C CNN
 	1    7350 8700
 	0    1    1    0
